File: kicad/board_connectors.kicad_sch (KiCad schematic)
At the start: 8 parts, among them J1001 RFShield_OnePiece, J1002 Conn_01x08, J1003 Conn_01x08, J1004 Conn_01x07, J1005 Conn_01x06, Q1003 PMCM4401VNE

Commit message: unify module and board
Parts:
- renumbered D1002 to D5, J1001 to J5, J1002 to J6, J1003 to J7, J1004 to J8, J1005 to J9, Q1003 to Q4, R1022 to R54
Changed lines of the file:
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@@
 		(on_board yes)
 		(dnp no)
-		(property "Reference" "#PWR01054"
+		(property "Reference" "#PWR0116"
 			(at 213.36 50.8 0)
 			(effects
@@
 			(project "riotee-module"
 				(path "/e235c9a3-080d-42b7-93df-883e69095a9f/1e27cf53-0710-4019-b3d0-1fa374a39b5a/71a24394-376e-48cc-9057-ddfdf0a39757/ceb14408-b4f4-4cc7-933c-90c2f9392878"
-					(reference "#PWR01054")
+					(reference "#PWR0116")
 					(unit 1)
 				)
@@
 		(dnp no)
 		(fields_autoplaced yes)
-		(property "Reference" "J1004"
+		(property "Reference" "J8"
 			(at 223.012 32.1853 0)
 			(effects
@@
 			(project "riotee-module"
 				(path "/e235c9a3-080d-42b7-93df-883e69095a9f/1e27cf53-0710-4019-b3d0-1fa374a39b5a/71a24394-376e-48cc-9057-ddfdf0a39757/ceb14408-b4f4-4cc7-933c-90c2f9392878"
-					(reference "J1004")
+					(reference "J8")
 					(unit 1)
 				)
@@
 		(on_board yes)
 		(dnp no)
-		(property "Reference" "R1022"
+		(property "Reference" "R54"
 			(at 150.368 68.6816 0)
 			(effects
@@
 			(project "riotee-module"
 				(path "/e235c9a3-080d-42b7-93df-883e69095a9f/1e27cf53-0710-4019-b3d0-1fa374a39b5a/71a24394-376e-48cc-9057-ddfdf0a39757/ceb14408-b4f4-4cc7-933c-90c2f9392878"
-					(reference "R1022")
+					(reference "R54")
 					(unit 1)
 				)
@@
 		(dnp no)
 		(fields_autoplaced yes)
-		(property "Reference" "J1003"
+		(property "Reference" "J7"
 			(at 217.17 100.4402 0)
 			(effects
@@
 			(project "riotee-module"
 				(path "/e235c9a3-080d-42b7-93df-883e69095a9f/1e27cf53-0710-4019-b3d0-1fa374a39b5a/71a24394-376e-48cc-9057-ddfdf0a39757/ceb14408-b4f4-4cc7-933c-90c2f9392878"
-					(reference "J1003")
+					(reference "J7")
 					(unit 1)
 				)
@@
 		(on_board yes)
 		(dnp no)
-		(property "Reference" "#PWR01050"
+		(property "Reference" "#PWR0112"
 			(at 87.63 157.48 0)
 			(effects
@@
 			(project "riotee-module"
 				(path "/e235c9a3-080d-42b7-93df-883e69095a9f/1e27cf53-0710-4019-b3d0-1fa374a39b5a/71a24394-376e-48cc-9057-ddfdf0a39757/ceb14408-b4f4-4cc7-933c-90c2f9392878"
-					(reference "#PWR01050")
+					(reference "#PWR0112")
 					(unit 1)
 				)
@@
 		(dnp no)
 		(fields_autoplaced yes)
-		(property "Reference" "Q1003"
+		(property "Reference" "Q4"
 			(at 162.687 63.9353 0)
 			(effects
@@
 			(project "riotee-module"
 				(path "/e235c9a3-080d-42b7-93df-883e69095a9f/1e27cf53-0710-4019-b3d0-1fa374a39b5a/71a24394-376e-48cc-9057-ddfdf0a39757/ceb14408-b4f4-4cc7-933c-90c2f9392878"
-					(reference "Q1003")
+					(reference "Q4")
 					(unit 1)
 				)
@@
 		(dnp no)
 		(fields_autoplaced yes)
-		(property "Reference" "J1002"
+		(property "Reference" "J6"
 			(at 194.31 100.4402 0)
 			(effects
@@
 			(project "riotee-module"
 				(path "/e235c9a3-080d-42b7-93df-883e69095a9f/1e27cf53-0710-4019-b3d0-1fa374a39b5a/71a24394-376e-48cc-9057-ddfdf0a39757/ceb14408-b4f4-4cc7-933c-90c2f9392878"
-					(reference "J1002")
+					(reference "J6")
 					(unit 1)
 				)
@@
 		(on_board yes)
 		(dnp no)
-		(property "Reference" "#PWR01052"
+		(property "Reference" "#PWR0114"
 			(at 160.02 83.82 0)
 			(effects
@@
 			(project "riotee-module"
 				(path "/e235c9a3-080d-42b7-93df-883e69095a9f/1e27cf53-0710-4019-b3d0-1fa374a39b5a/71a24394-376e-48cc-9057-ddfdf0a39757/ceb14408-b4f4-4cc7-933c-90c2f9392878"
-					(reference "#PWR01052")
+					(reference "#PWR0114")
 					(unit 1)
 				)
@@
 		(dnp no)
 		(fields_autoplaced yes)
-		(property "Reference" "J1001"
+		(property "Reference" "J5"
 			(at 103.632 137.5953 0)
 			(effects
@@
 			(project "riotee-module"
 				(path "/e235c9a3-080d-42b7-93df-883e69095a9f/1e27cf53-0710-4019-b3d0-1fa374a39b5a/71a24394-376e-48cc-9057-ddfdf0a39757/ceb14408-b4f4-4cc7-933c-90c2f9392878"
-					(reference "J1001")
+					(reference "J5")
 					(unit 1)
 				)
@@
 		(on_board yes)
 		(dnp no)
-		(property "Reference" "#PWR01056"
+		(property "Reference" "#PWR0118"
 			(at 224.79 132.08 0)
 			(effects
@@
 			(project "riotee-module"
 				(path "/e235c9a3-080d-42b7-93df-883e69095a9f/1e27cf53-0710-4019-b3d0-1fa374a39b5a/71a24394-376e-48cc-9057-ddfdf0a39757/ceb14408-b4f4-4cc7-933c-90c2f9392878"
-					(reference "#PWR01056")
+					(reference "#PWR0118")
 					(unit 1)
 				)
@@
 		(dnp no)
 		(fields_autoplaced yes)
-		(property "Reference" "J1005"
+		(property "Reference" "J9"
 			(at 220.98 62.3402 0)
 			(effects
@@
 			(project "riotee-module"
 				(path "/e235c9a3-080d-42b7-93df-883e69095a9f/1e27cf53-0710-4019-b3d0-1fa374a39b5a/71a24394-376e-48cc-9057-ddfdf0a39757/ceb14408-b4f4-4cc7-933c-90c2f9392878"
-					(reference "J1005")
+					(reference "J9")
 					(unit 1)
 				)
@@
 		(on_board yes)
 		(dnp no)
-		(property "Reference" "D1002"
+		(property "Reference" "D5"
 			(at 154.5082 50.9778 0)
 			(effects
@@
 			(project "riotee-module"
 				(path "/e235c9a3-080d-42b7-93df-883e69095a9f/1e27cf53-0710-4019-b3d0-1fa374a39b5a/71a24394-376e-48cc-9057-ddfdf0a39757/ceb14408-b4f4-4cc7-933c-90c2f9392878"
-					(reference "D1002")
+					(reference "D5")
 					(unit 1)
 				)
@@
 		(on_board yes)
 		(dnp no)
-		(property "Reference" "#PWR01051"
+		(property "Reference" "#PWR0113"
 			(at 160.02 48.26 0)
 			(effects
@@
 			(project "riotee-module"
 				(path "/e235c9a3-080d-42b7-93df-883e69095a9f/1e27cf53-0710-4019-b3d0-1fa374a39b5a/71a24394-376e-48cc-9057-ddfdf0a39757/ceb14408-b4f4-4cc7-933c-90c2f9392878"
-					(reference "#PWR01051")
+					(reference "#PWR0113")
 					(unit 1)
 				)
@@
 		(on_board yes)
 		(dnp no)
-		(property "Reference" "#PWR01055"
+		(property "Reference" "#PWR0117"
 			(at 224.79 101.6 0)
 			(effects
@@
 			(project "riotee-module"
 				(path "/e235c9a3-080d-42b7-93df-883e69095a9f/1e27cf53-0710-4019-b3d0-1fa374a39b5a/71a24394-376e-48cc-9057-ddfdf0a39757/ceb14408-b4f4-4cc7-933c-90c2f9392878"
-					(reference "#PWR01055")
+					(reference "#PWR0117")
 					(unit 1)
 				)
@@
 		(on_board yes)
 		(dnp no)
-		(property "Reference" "#PWR01053"
+		(property "Reference" "#PWR0115"
 			(at 186.69 133.35 0)
 			(effects
@@
 			(project "riotee-module"
 				(path "/e235c9a3-080d-42b7-93df-883e69095a9f/1e27cf53-0710-4019-b3d0-1fa374a39b5a/71a24394-376e-48cc-9057-ddfdf0a39757/ceb14408-b4f4-4cc7-933c-90c2f9392878"
-					(reference "#PWR01053")
-					(unit 1)
-				)
+					(reference "#PWR0115")
+					(unit 1)
+				)
