File: kicad/usb_power.kicad_sch (KiCad schematic)
At the start: 11 parts, among them J1 12402012E212A, U7 TLV73333PDBV, U8 TPS71721DCK

Commit message: copy in module schematics
Changed lines of the file:
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@@
 (kicad_sch
-	(version 20231120)
+	(version 20250114)
 	(generator "eeschema")
-	(generator_version "8.0")
+	(generator_version "9.0")
 	(paper "A4")
 	(junction
@@
 	(label "USB.D-"
 		(at 102.87 92.71 0)
-		(fields_autoplaced yes)
 		(effects
 			(font
@@
 	(label "USB.D+"
 		(at 102.87 97.79 0)
-		(fields_autoplaced yes)
 		(effects
 			(font
@@
 		(shape input)
 		(at 124.46 90.17 0)
-		(fields_autoplaced yes)
 		(effects
 			(font
