File: kicad/module_connection.kicad_sch (KiCad schematic)
At the start: 13 parts, among them J2 Conn_01x12, J3 Conn_01x10, J4 Conn_01x02, Q1 SI2302CDS, SW1 CNK_KMR2, U9 TS5A3166YZP

Commit message: unify module and board
Connections:
- net SCL renamed SYS.SCL
- net SDA renamed SYS.SDA
- net TargetVcc renamed VCC
Other:
- sheet Module renamed Riotee Module
- sheet Riotee Module ports: added BYPASS_SHUNT, D[0..10], EN_BUCK, SBW{CLK,IO}, SWD{CLK,IO}, SYS{SCL,SDA}, VBUCK, VCAP, VCAP_SENSE, VSHUNT, VSRC; removed none
- moved on the sheet: J4

Commit message: resolve ERC
Connections:
- net A0 renamed D2
- net A1 renamed D3
