File: kicad/energy_management.kicad_sch (KiCad schematic)
At the start: 23 parts, among them U1003 TLV369DCK, U1004 TLV7032

Commit message: unify module and board
Parts:
- renumbered C1009 to C41, C1010 to C42, C1011 to C43, C1012 to C44, C1013 to C45, R1005 to R38, R1006 to R39, R1007 to R40, R1008 to R41, R1009 to R42, R1010 to R43, R1011 to R44, R1012 to R45, R1013 to R46, R1014 to R47, R1015 to R48, R1016 to R49, R1017 to R50, R1018 to R51, R1019 to R52, R1020 to R53, U1003 to U13, U1004 to U14

Commit message: move module parts to common library
Parts:
- U13: symbol Riotee:TLV369DCK -> riotee:TLV369DCK
- U14: symbol Riotee:TLV7032 -> riotee:TLV7032
Changed lines of the file:
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@@
 	)
 	(symbol
-		(lib_id "Riotee:TLV7032")
+		(lib_id "riotee:TLV7032")
 		(at 217.17 96.52 0)
 		(unit 1)
@@
 			)
 		)
-		(property "Description" "Dual comparator, Iq=315nA/Ch"
+		(property "Description" "Dual, 1.8V Low Power, Rail-to-Rail Input, Push-Pull Output Comparator, DSBGA-8"
 			(at 217.17 96.52 0)
 			(effects
@@
 	)
 	(symbol
-		(lib_id "Riotee:TLV7032")
+		(lib_id "riotee:TLV7032")
 		(at 226.06 114.3 0)
 		(unit 2)
@@
 	)
 	(symbol
-		(lib_id "Riotee:TLV7032")
+		(lib_id "riotee:TLV7032")
 		(at 217.17 96.52 0)
 		(unit 3)
@@
 			)
 		)
-		(property "Description" "Dual comparator, Iq=315nA/Ch"
+		(property "Description" "Dual, 1.8V Low Power, Rail-to-Rail Input, Push-Pull Output Comparator, DSBGA-8"
 			(at 217.17 96.52 0)
 			(effects
@@
 	)
 	(symbol
-		(lib_id "Riotee:TLV369DCK")
+		(lib_id "riotee:TLV369DCK")
 		(at 74.93 64.77 0)
 		(unit 1)
@@
 			)
 		)
-		(property "Datasheet" ""
+		(property "Datasheet" "http://www.ti.com/lit/ds/symlink/lm321.pdf"
 			(at 74.93 64.77 0)
 			(effects
@@
 			)
 		)
-		(property "Description" "Op-Amp, Iq=800nA"
+		(property "Description" "Low Power Single Operational Amplifier, SOT-23-5"
 			(at 74.93 64.77 0)
 			(effects

Commit message: resolve ERC
Parts:
- C41, C42, C43, C44, C45: footprint Riotee:C_0201_0603Metric -> riotee:C_0201_0603Metric; symbol Riotee:C -> Device:C
- R38, R39, R40, R41, R42, R43, R44, R45, R46, R47, R48, R49, R50, R51, R52, R53: footprint Riotee:R_0201_0603Metric -> riotee:R_0201_0603Metric; symbol Riotee:R -> Device:R
- U13: footprint Riotee:TI_SC70-5_DCK5 -> riotee:TI_SC70-5_DCK5
- U14: footprint Riotee:TI_WSON8_DSG -> riotee:TI_WSON8_DSG

Commit message: resolve remaining import errors
Parts:
- C41, C42, C43, C44, C45: footprint riotee:C_0201_0603Metric -> Capacitor_SMD:C_0201_0603Metric
- R38, R39, R40, R41, R42, R43, R44, R45, R46, R47, R48, R49, R50, R51, R52, R53: footprint riotee:R_0201_0603Metric -> Resistor_SMD:R_0201_0603Metric
Changed lines of the file:
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@@
 			)
 		)
-		(property "Footprint" "riotee:R_0201_0603Metric"
+		(property "Footprint" "Resistor_SMD:R_0201_0603Metric"
 			(at 64.77 166.878 90)
 			(effects
@@
 			)
 		)
-		(property "Footprint" "riotee:R_0201_0603Metric"
+		(property "Footprint" "Resistor_SMD:R_0201_0603Metric"
 			(at 78.74 80.772 90)
 			(effects
@@
 			)
 		)
-		(property "Footprint" "riotee:R_0201_0603Metric"
+		(property "Footprint" "Resistor_SMD:R_0201_0603Metric"
 			(at 126.492 139.7 90)
 			(effects
@@
 			)
 		)
-		(property "Footprint" "riotee:R_0201_0603Metric"
+		(property "Footprint" "Resistor_SMD:R_0201_0603Metric"
 			(at 126.492 160.02 90)
 			(effects
@@
 			)
 		)
-		(property "Footprint" "riotee:R_0201_0603Metric"
+		(property "Footprint" "Resistor_SMD:R_0201_0603Metric"
 			(at 120.65 156.718 90)
 			(effects
@@
 			)
 		)
-		(property "Footprint" "riotee:R_0201_0603Metric"
+		(property "Footprint" "Resistor_SMD:R_0201_0603Metric"
 			(at 70.612 149.86 90)
 			(effects
@@
 			)
 		)
-		(property "Footprint" "riotee:C_0201_0603Metric"
+		(property "Footprint" "Capacitor_SMD:C_0201_0603Metric"
 			(at 142.5448 154.94 0)
 			(effects
@@
 			)
 		)
-		(property "Footprint" "riotee:R_0201_0603Metric"
+		(property "Footprint" "Resistor_SMD:R_0201_0603Metric"
 			(at 120.65 166.878 90)
 			(effects
@@
 			)
 		)
-		(property "Footprint" "riotee:R_0201_0603Metric"
+		(property "Footprint" "Resistor_SMD:R_0201_0603Metric"
 			(at 55.372 54.61 90)
 			(effects
@@
 			)
 		)
-		(property "Footprint" "riotee:R_0201_0603Metric"
+		(property "Footprint" "Resistor_SMD:R_0201_0603Metric"
 			(at 88.9 62.992 90)
 			(effects
@@
 			)
 		)
-		(property "Footprint" "riotee:C_0201_0603Metric"
+		(property "Footprint" "Capacitor_SMD:C_0201_0603Metric"
 			(at 207.3148 74.93 0)
 			(effects
@@
 			)
 		)
-		(property "Footprint" "riotee:R_0201_0603Metric"
+		(property "Footprint" "Resistor_SMD:R_0201_0603Metric"
 			(at 70.612 170.18 90)
 			(effects
@@
 			)
 		)
-		(property "Footprint" "riotee:R_0201_0603Metric"
+		(property "Footprint" "Resistor_SMD:R_0201_0603Metric"
 			(at 55.372 72.39 90)
 			(effects
@@
 			)
 		)
-		(property "Footprint" "riotee:R_0201_0603Metric"
+		(property "Footprint" "Resistor_SMD:R_0201_0603Metric"
 			(at 70.612 160.02 90)
 			(effects
@@
 			)
 		)
-		(property "Footprint" "riotee:C_0201_0603Metric"
+		(property "Footprint" "Capacitor_SMD:C_0201_0603Metric"
 			(at 86.6648 154.94 0)
 			(effects
@@
 			)
 		)
-		(property "Footprint" "riotee:C_0201_0603Metric"
+		(property "Footprint" "Capacitor_SMD:C_0201_0603Metric"
 			(at 74.93 74.6252 0)
 			(effects
@@
 			)
 		)
-		(property "Footprint" "riotee:R_0201_0603Metric"
+		(property "Footprint" "Resistor_SMD:R_0201_0603Metric"
 			(at 126.492 149.86 90)
 			(effects
@@
 			)
 		)
-		(property "Footprint" "riotee:R_0201_0603Metric"
+		(property "Footprint" "Resistor_SMD:R_0201_0603Metric"
 			(at 70.612 139.7 90)
 			(effects
@@
 			)
 		)
-		(property "Footprint" "riotee:R_0201_0603Metric"
+		(property "Footprint" "Resistor_SMD:R_0201_0603Metric"
 			(at 126.492 170.18 90)
 			(effects
@@
 			)
 		)
-		(property "Footprint" "riotee:R_0201_0603Metric"
+		(property "Footprint" "Resistor_SMD:R_0201_0603Metric"
 			(at 64.77 156.718 90)
 			(effects
@@
 			)
 		)
-		(property "Footprint" "riotee:C_0201_0603Metric"
+		(property "Footprint" "Capacitor_SMD:C_0201_0603Metric"
 			(at 77.7748 40.64 0)
 			(effects
